File: hw/boards/io_wrapper_board/io_wrapper_board.kicad_sch (KiCad schematic)
At the start: 0 parts

Commit message: 147 - [hw/boards/io_wrapper_board/] 1st draft of io wrapper board
Parts:
- added J1: DIN41612_02x16_AB, f4bjh_ICs:DIN41612_B2_2x16_Male_Horizontal_THT, symbol f4bjh_ICs:DIN41612_02x16_AB
- added J2: Conn_01x16, f4bjh_ICs:IDC-Header_2x08_P2.54mm_Vertical, symbol Connector_Generic:Conn_01x16
- added J3: Conn_01x02, TerminalBlock:TerminalBlock_Xinya_XY308-2.54-2P_1x02_P2.54mm_Horizontal, symbol Connector_Generic:Conn_01x02
Connections:
- new net: J1.b7 (Pin_b7), J2.10 (Pin_10)
- new net: J1.b9 (Pin_b9), J2.11 (Pin_11)
- new net: J1.b11 (Pin_b11), J2.14 (Pin_14)
- new net: J1.b13 (Pin_b13), J2.15 (Pin_15)
- new net: J1.a13 (Pin_a13), J2.2 (Pin_2)
- new net: J1.a11 (Pin_a11), J2.3 (Pin_3)
- new net: J1.a9 (Pin_a9), J2.6 (Pin_6)
- new net: J1.a7 (Pin_a7), J2.7 (Pin_7)
- new net: J1.a5 (Pin_a5), J2.8 (Pin_8)
- new net: J1.b5 (Pin_b5), J2.9 (Pin_9)
- new net +5V: J1.a15 (Pin_a15), J1.a2 (Pin_a2), J1.a3 (Pin_a3), J1.b15 (Pin_b15), J1.b2 (Pin_b2), J1.b3 (Pin_b3), J3.1 (Pin_1)
- new net GND: J1.a1 (Pin_a1), J1.a10 (Pin_a10), J1.a12 (Pin_a12), J1.a14 (Pin_a14), J1.a16 (Pin_a16), J1.a4 (Pin_a4), J1.a6 (Pin_a6), J1.a8 (Pin_a8), J1.b1 (Pin_b1), J1.b10 (Pin_b10), J1.b12 (Pin_b12), J1.b14 (Pin_b14), J1.b16 (Pin_b16), J1.b4 (Pin_b4), J1.b6 (Pin_b6), J1.b8 (Pin_b8), J2.1 (Pin_1), J2.12 (Pin_12), J2.13 (Pin_13), J2.16 (Pin_16), J2.4 (Pin_4), J2.5 (Pin_5), J3.2 (Pin_2)
