File: hw/boards/backplane_board/backplane_board.kicad_pcb (KiCad board)
At the start: 2 copper layers, 4 parts, among them J1 DIN41612_02x16_AB, J2 DIN41612_02x16_AB, J3 DIN41612_02x16_AB, J4 DIN41612_02x16_AB

Commit message: 147 - [hw/boards/backplane_board/] ajoute le contour du PCB
Other:
- board outline added: 290.8 x 56.7 mm
Changed lines of the file:
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@@
 		)
+	)
+	(gr_rect
+		(start -19.05 71.55)
+		(end 271.78 128.27)
+		(stroke
+			(width 0.05)
+			(type default)
+		)
+		(fill no)
+		(layer "Edge.Cuts")
 	)
 	(segment
@@
 	)
 	(segment
+		(start 162.54 82.54)
+		(end 160 82.54)
+		(width 1.5)
+		(layer "F.Cu")
+		(net 3)
+	)
+	(segment
 		(start 92.54 82.54)
 		(end 160 82.54)
@@
 	)
 	(segment
-		(start 160 82.54)
-		(end 162.54 82.54)
+		(start 162.54 115.56)
+		(end 160 115.56)
 		(width 1.5)
 		(layer "F.Cu")
@@
 		(width 1.5)
 		(layer "F.Cu")
-		(net 3)
-	)
-	(segment
-		(start 160 115.56)
-		(end 162.54 115.56)
-		(width 1.5)
-		(layer "F.Cu")
